File: mockingboard2k.kicad_pcb (KiCad board)
At the start: 2 copper layers, 130.9 x 78.2 mm, 33 parts, among them J1 AUDIO_OUT, P1 A2Bus, U1 AY-3-8910, U2 6522, U3 74HCT74, U4 74AHCT1G04, U5 AY-3-8910, U6 6522

Commit message: Version 1 ordered at JLCPCB
Connections:
- U3 pad 2: PHI0 -> Net-(U3-Pad12)
- U3 pad 3: 7M -> unconnected-(U3-Pad3)
- U3 pad 5: Net-(U3-Pad12) -> PHI0
Routing:
- net PHI0: track 46.2 -> 52.6 mm
- net Net-(U3-Pad12): track 6.33 -> 0.00 mm
Other:
- board text added: "Version 1"

Commit message: Tweaks
Connections:
- U3 pad 2: Net-(U3-Pad12) -> PHI0
- U3 pad 3: unconnected-(U3-Pad3) -> 7M
- U3 pad 5: PHI0 -> Net-(U3-Pad12)
Routing:
- net PHI0: track 52.6 -> 46.2 mm
- net Net-(U3-Pad12): track 0.00 -> 6.33 mm
Other:
- board text added: "Version 2"
- board text removed: "Version 1"
Changed lines of the file:
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@@
   (net 142 "unconnected-(U5-Pad39)")
   (net 143 "unconnected-(U6-Pad39)")
-  (net 144 "unconnected-(U3-Pad3)")
   (footprint "apple2-bus:Male_Card-Edge_50_pin__100_mil" (layer "F.Cu")
     (at 167.259 139.446)
@@
       (net 30 "PHI0") (pinfunction "~{R}") (pintype "input"))
     (pad "2" smd roundrect (at -2.8625 1.3) (size 1.475 0.4) (layers "B.Cu" "B.Paste" "B.Mask") (roundrect_rratio 0.25)
-      (net 20 "Net-(U3-Pad12)") (pinfunction "D") (pintype "input"))
+      (net 30 "PHI0") (pinfunction "D") (pintype "input"))
     (pad "3" smd roundrect (at -2.8625 0.65) (size 1.475 0.4) (layers "B.Cu" "B.Paste" "B.Mask") (roundrect_rratio 0.25)
-      (net 144 "unconnected-(U3-Pad3)") (pinfunction "C") (pintype "input"))
+      (net 3 "7M") (pinfunction "C") (pintype "input"))
     (pad "4" smd roundrect (at -2.8625 0) (size 1.475 0.4) (layers "B.Cu" "B.Paste" "B.Mask") (roundrect_rratio 0.25)
       (net 15 "VCC") (pinfunction "~{S}") (pintype "input"))
     (pad "5" smd roundrect (at -2.8625 -0.65) (size 1.475 0.4) (layers "B.Cu" "B.Paste" "B.Mask") (roundrect_rratio 0.25)
-      (net 30 "PHI0") (pinfunction "Q") (pintype "output"))
+      (net 20 "Net-(U3-Pad12)") (pinfunction "Q") (pintype "output"))
     (pad "6" smd roundrect (at -2.8625 -1.3) (size 1.475 0.4) (layers "B.Cu" "B.Paste" "B.Mask") (roundrect_rratio 0.25)
-      (net 22 "unconnected-(U3-Pad6)") (pinfunction "~{Q}") (pintype "output"))
+      (net 22 "unconnected-(U3-Pad6)") (pinfunction "~{Q}") (pintype "output+no_connect"))
     (pad "7" smd roundrect (at -2.8625 -1.95) (size 1.475 0.4) (layers "B.Cu" "B.Paste" "B.Mask") (roundrect_rratio 0.25)
       (net 16 "GND") (pinfunction "GND") (pintype "power_in"))
@@
   (gr_line (start 78.105 65.024) (end 75.692 67.437) (layer "Edge.Cuts") (width 0.15))
   (gr_line (start 206.629 67.31) (end 204.343 65.024) (layer "Edge.Cuts") (width 0.15))
-  (gr_text "Version 1" (at 142.24 73.152) (layer "F.SilkS")
+  (gr_text "GND" (at 198.247 72.39 90) (layer "F.SilkS")
+    (effects (font (size 1 1) (thickness 0.15)) (justify left))
+  )
+  (gr_text "Version 2" (at 142.24 73.152) (layer "F.SilkS")
     (effects (font (size 1.5 1.5) (thickness 0.3)))
   )
@@
     (effects (font (size 6 4) (thickness 0.75)) (justify left))
   )
+  (gr_text "RIGHT" (at 203.327 72.39 90) (layer "F.SilkS")
+    (effects (font (size 1 1) (thickness 0.15)) (justify left))
+  )
   (gr_text "https://github.com/hanshuebner/mockingboard2k" (at 81.915 128.905) (layer "F.SilkS")
     (effects (font (size 3 2) (thickness 0.35)) (justify left))
   )
-  (gr_text "GND" (at 198.247 72.39 90) (layer "F.Mask")
+  (gr_text "LEFT" (at 195.834 72.39 90) (layer "F.SilkS")
     (effects (font (size 1 1) (thickness 0.15)) (justify left))
   )
-  (gr_text "RIGHT" (at 203.327 72.39 90) (layer "F.Mask")
-    (effects (font (size 1 1) (thickness 0.15)) (justify left))
-  )
-  (gr_text "LEFT" (at 195.834 72.39 90) (layer "F.Mask")
-    (effects (font (size 1 1) (thickness 0.15)) (justify left))
-  )
-  (gr_text "GND" (at 200.787 72.39 90) (layer "F.Mask")
+  (gr_text "GND" (at 200.787 72.39 90) (layer "F.SilkS")
     (effects (font (size 1 1) (thickness 0.15)) (justify left))
   )
@@
   (segment (start 179.824981 80.872514) (end 179.832 80.865495) (width 0.25) (layer "B.Cu") (net 19))
   (segment (start 179.832 80.865495) (end 179.832 78.232) (width 0.25) (layer "B.Cu") (net 19))
+  (segment (start 174.461804 107.3) (end 173.6675 107.3) (width 0.25) (layer "B.Cu") (net 20))
+  (segment (start 179.3925 108.6) (end 179.317999 108.674501) (width 0.25) (layer "B.Cu") (net 20))
+  (segment (start 179.317999 108.674501) (end 175.836305 108.674501) (width 0.25) (layer "B.Cu") (net 20))
+  (segment (start 175.836305 108.674501) (end 174.461804 107.3) (width 0.25) (layer "B.Cu") (net 20))
   (segment (start 158.75 123.952) (end 145.415 123.952) (width 0.25) (layer "F.Cu") (net 21))
   (segment (start 141.6945 123.19) (end 85.979 123.19) (width 0.25) (layer "F.Cu") (net 21))
@@
   (via (at 163.322 109.22) (size 0.8) (drill 0.4) (layers "F.Cu" "B.Cu") (net 30))
   (via (at 172.885895 109.384496) (size 0.8) (drill 0.4) (layers "F.Cu" "B.Cu") (net 30))
-  (segment (start 174.461804 107.3) (end 173.6675 107.3) (width 0.25) (layer "B.Cu") (net 30))
-  (segment (start 179.3925 108.6) (end 179.317999 108.674501) (width 0.25) (layer "B.Cu") (net 30))
   (segment (start 162.179 137.033) (end 163.322 135.89) (width 0.25) (layer "B.Cu") (net 30))
   (segment (start 173.6675 109.25) (end 173.6675 109.9) (width 0.25) (layer "B.Cu") (net 30))
-  (segment (start 179.317999 108.674501) (end 175.836305 108.674501) (width 0.25) (layer "B.Cu") (net 30))
-  (segment (start 175.836305 108.674501) (end 174.461804 107.3) (width 0.25) (layer "B.Cu") (net 30))
   (segment (start 162.179 139.446) (end 162.179 137.033) (width 0.25) (layer "B.Cu") (net 30))
   (segment (start 179.317011 109.325489) (end 179.3925 109.25) (width 0.25) (layer "B.Cu") (net 30))

Commit message: 6522A(!)
Parts:
- U2, U6: value 6522 -> 6522A
Changed lines of the file:
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@@
       (effects (font (size 1 1) (thickness 0.15)))
     )
-    (fp_text value "6522" (at 9.19 24.178358) (layer "F.SilkS")
+    (fp_text value "6522A" (at 9.19 24.178358) (layer "F.SilkS")
       (effects (font (size 1 1) (thickness 0.15)))
     )
@@
       (effects (font (size 1 1) (thickness 0.15)))
     )
-    (fp_text value "6522" (at 9.317 24.178358 180) (layer "F.SilkS")
-      (effects (font (size 1 1) (thickness 0.15)))
-    )
+    (fp_text value "6522A" (at 9.317 24.178358 180) (layer "F.SilkS")
+      (effects (font (size 1 1) (thickness 0.15)))
+    )
