File: mockingboard2k.kicad_sch (KiCad schematic)
At the start: 33 parts, among them J1 AUDIO_OUT, P1 A2Bus, U1 AY-3-8910, U2 6522, U3 74HCT74, U4 74AHCT1G04, U5 AY-3-8910, U6 6522

Commit message: Version 1 ordered at JLCPCB
Parts:
- C1, C2: LCSC (none) -> C2835555
- C3, C4, C5, C6, C7, C8, C9: LCSC (none) -> C2830722
- D1, D2, D3, D4: LCSC (none) -> C77343
- R1, R2, R3, R7, R8, R9: LCSC (none) -> C325761
- R10, R11, R12, R4, R5, R6: LCSC (none) -> C269542
- U3: LCSC (none) -> C8164
- U4: LCSC (none) -> C460498
Connections:
- net 7M: no longer U3.3 (C)
- net PHI0: now also U3.5 (Q); no longer U3.2 (D)
- net at U3.12 (D): now also U3.2 (D); no longer U3.5 (Q)
Changed lines of the file:
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@@
+      (effects (font (size 1.27 1.27)) hide)
+    )
+    (property "LCSC" "C2830722" (id 15) (at 59.69 229.235 0)
       (effects (font (size 1.27 1.27)) hide)
     )
@@
       (effects (font (size 1.27 1.27)) hide)
     )
+    (property "LCSC" "C2830722" (id 15) (at 64.77 229.235 0)
+      (effects (font (size 1.27 1.27)) hide)
+    )
     (pin "1")
     (pin "2")
@@
       (effects (font (size 1.27 1.27)) hide)
     )
+    (property "LCSC" "C2830722" (id 15) (at 69.85 229.235 0)
+      (effects (font (size 1.27 1.27)) hide)
+    )
     (pin "1")
     (pin "2")
@@
       (effects (font (size 1.27 1.27)) hide)
     )
+    (property "LCSC" "C2830722" (id 15) (at 74.93 229.235 0)
+      (effects (font (size 1.27 1.27)) hide)
+    )
     (pin "1")
     (pin "2")
@@
     )
     (property "Vendor 2 URL" "https://www.digikey.com/products/en?keywords=1276-1286-1-ND" (id 14) (at 8.89 401.955 0)
+      (effects (font (size 1.27 1.27)) hide)
+    )
+    (property "LCSC" "C2830722" (id 15) (at 80.01 229.235 0)
       (effects (font (size 1.27 1.27)) hide)
     )
@@
       (effects (font (size 1.27 1.27)) hide)
     )
+    (property "LCSC" "C2830722" (id 15) (at 49.53 229.235 0)
+      (effects (font (size 1.27 1.27)) hide)
+    )
     (pin "1")
     (pin "2")
@@
     )
     (property "Vendor 2 URL" "https://www.digikey.com/products/en?keywords=1276-1286-1-ND" (id 14) (at 8.89 401.955 0)
+      (effects (font (size 1.27 1.27)) hide)
+    )
+    (property "LCSC" "C2830722" (id 15) (at 54.61 229.235 0)
       (effects (font (size 1.27 1.27)) hide)
     )
@@
       (effects (font (size 1.27 1.27)) hide)
     )
+    (property "LCSC" "C77343" (id 15) (at 177.8 173.355 0)
+      (effects (font (size 1.27 1.27)) hide)
+    )
     (pin "1")
     (pin "2")
@@
       (effects (font (size 1.27 1.27)) hide)
     )
+    (property "LCSC" "C77343" (id 15) (at 177.8 80.01 0)
+      (effects (font (size 1.27 1.27)) hide)
+    )
     (pin "1")
     (pin "2")
@@
     )
     (property "Datasheet" "~" (id 3) (at 294.64 225.425 0)
+      (effects (font (size 1.27 1.27)) hide)
+    )
+    (property "LCSC" "C269542" (id 15) (at 297.18 155.575 0)
       (effects (font (size 1.27 1.27)) hide)
     )
@@
       (effects (font (size 1.27 1.27)) hide)
     )
+    (property "LCSC" "C2835555" (id 4) (at 314.96 123.19 90)
+      (effects (font (size 1.27 1.27)) hide)
+    )
     (pin "1")
     (pin "2")
@@
       (effects (font (size 1.27 1.27)) hide)
     )
+    (property "LCSC" "C325761" (id 15) (at 297.18 155.575 0)
+      (effects (font (size 1.27 1.27)) hide)
+    )
     (pin "1")
     (pin "2")
@@
     )
     (property "Datasheet" "~" (id 3) (at 304.8 213.995 0)
+      (effects (font (size 1.27 1.27)) hide)
+    )
+    (property "LCSC" "C325761" (id 15) (at 297.18 155.575 0)
       (effects (font (size 1.27 1.27)) hide)
     )
@@
       (effects (font (size 1.27 1.27)) hide)
     )
+    (property "LCSC" "C460498" (id 4) (at 149.86 180.975 0)
+      (effects (font (size 1.27 1.27)) hide)
+    )
     (pin "2")
     (pin "3")
@@
       (effects (font (size 1.27 1.27)) hide)
     )
+    (property "LCSC" "C77343" (id 15) (at 297.18 155.575 0)
+      (effects (font (size 1.27 1.27)) hide)
+    )
     (pin "1")
     (pin "2")
@@
       (effects (font (size 1.27 1.27)) hide)
     )
+    (property "LCSC" "C77343" (id 15) (at 297.18 62.23 0)
+      (effects (font (size 1.27 1.27)) hide)
+    )
     (pin "1")
     (pin "2")
@@
       (effects (font (size 1.27 1.27)) hide)
     )
+    (property "LCSC" "C269542" (id 15) (at 297.18 155.575 0)
+      (effects (font (size 1.27 1.27)) hide)
+    )
     (pin "1")
     (pin "2")
@@
       (effects (font (size 1.27 1.27)) hide)
     )
+    (property "LCSC" "C269542" (id 15) (at 297.18 155.575 0)
+      (effects (font (size 1.27 1.27)) hide)
+    )
     (pin "1")
     (pin "2")
@@
     )
     (property "Datasheet" "~" (id 3) (at 304.8 219.075 0)
+      (effects (font (size 1.27 1.27)) hide)
+    )
+    (property "LCSC" "C325761" (id 15) (at 297.18 155.575 0)
       (effects (font (size 1.27 1.27)) hide)
     )
@@
       (effects (font (size 1.27 1.27)) hide)
     )
+    (property "LCSC" "C2835555" (id 4) (at 314.96 216.535 90)
+      (effects (font (size 1.27 1.27)) hide)
+    )
     (pin "1")
     (pin "2")
@@
       (effects (font (size 1.27 1.27)) hide)
     )
+    (property "LCSC" "C269542" (id 15) (at 297.18 155.575 0)
+      (effects (font (size 1.27 1.27)) hide)
+    )
     (pin "1")
     (pin "2")
@@
       (effects (font (size 1.27 1.27)) hide)
     )
+    (property "LCSC" "C269542" (id 15) (at 297.18 155.575 0)
+      (effects (font (size 1.27 1.27)) hide)
+    )
     (pin "1")
     (pin "2")
@@
     (pin "1")
   )
-  (symbol (lib_id "74xx:74LS74") (at 71.12 180.34 0) (unit 1)
+  (symbol (lib_id "74xx:74LS74") (at 71.12 180.34 0) (mirror y) (unit 1)
     (in_bom yes) (on_board yes) (fields_autoplaced)
-    (property "Reference" "U3" (id 0) (at 73.1394 171.5602 0)
-      (effects (font (size 1.27 1.27)) (justify left))
-    )
-    (property "Value" "74HCT74" (id 1) (at 73.1394 174.0971 0)
-      (effects (font (size 1.27 1.27)) (justify left))
+    (property "Reference" "U3" (id 0) (at 71.6406 171.5602 0)
+      (effects (font (size 1.27 1.27)) (justify right))
+    )
+    (property "Value" "74HCT74" (id 1) (at 71.6406 174.0971 0)
+      (effects (font (size 1.27 1.27)) (justify right))
     )
     (property "Footprint" "Package_SO:TSSOP-14_4.4x5mm_P0.65mm" (id 2) (at 71.12 180.34 0)
@@
     )
     (property "Datasheet" "74xx/74hc_hct74.pdf" (id 3) (at 71.12 180.34 0)
+      (effects (font (size 1.27 1.27)) hide)
+    )
+    (property "LCSC" "C8164" (id 4) (at 71.12 180.34 0)
       (effects (font (size 1.27 1.27)) hide)
     )
@@
       (effects (font (size 1.27 1.27)) hide)
     )
+    (property "LCSC" "C325761" (id 15) (at 297.18 155.575 0)
+      (effects (font (size 1.27 1.27)) hide)
+    )
     (pin "1")
     (pin "2")
@@
       (effects (font (size 1.27 1.27)) hide)
     )
+    (property "LCSC" "C269542" (id 15) (at 297.18 155.575 0)
+      (effects (font (size 1.27 1.27)) hide)
+    )
     (pin "1")
     (pin "2")
@@
     )
     (property "Datasheet" "74xx/74hc_hct74.pdf" (id 3) (at 94.615 180.34 0)
+      (effects (font (size 1.27 1.27)) hide)
+    )
+    (property "LCSC" "C8164" (id 4) (at 94.615 180.34 0)
       (effects (font (size 1.27 1.27)) hide)
     )
@@
       (effects (font (size 1.27 1.27)) hide)
     )
+    (property "LCSC" "C325761" (id 15) (at 297.18 155.575 0)
+      (effects (font (size 1.27 1.27)) hide)
+    )
     (pin "1")
     (pin "2")
@@
       (effects (font (size 1.27 1.27)) hide)
     )
+    (property "LCSC" "C325761" (id 15) (at 297.18 155.575 0)
+      (effects (font (size 1.27 1.27)) hide)
+    )

Commit message: Tweaks
Connections:
- net 7M: now also U3.3 (C)
- net PHI0: now also U3.2 (D); no longer U3.5 (Q)
- net at U3.12 (D): now also U3.5 (Q); no longer U3.2 (D)
- no-connect marks 76 -> 75
Changed lines of the file:
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@@
   (no_connect (at 100.33 76.2))
   (no_connect (at 78.74 182.88))
-  (no_connect (at 99.06 173.99))
   (no_connect (at 185.42 125.73))
   (wire (pts (xy 288.29 68.58) (xy 302.26 68.58))
@@
     (pin "1")
   )
-  (symbol (lib_id "74xx:74LS74") (at 71.12 180.34 0) (mirror y) (unit 1)
+  (symbol (lib_id "74xx:74LS74") (at 71.12 180.34 0) (unit 1)
     (in_bom yes) (on_board yes) (fields_autoplaced)
-    (property "Reference" "U3" (id 0) (at 71.6406 171.5602 0)
-      (effects (font (size 1.27 1.27)) (justify right))
-    )
-    (property "Value" "74HCT74" (id 1) (at 71.6406 174.0971 0)
-      (effects (font (size 1.27 1.27)) (justify right))
+    (property "Reference" "U3" (id 0) (at 73.1394 171.5602 0)
+      (effects (font (size 1.27 1.27)) (justify left))
+    )
+    (property "Value" "74HCT74" (id 1) (at 73.1394 174.0971 0)
+      (effects (font (size 1.27 1.27)) (justify left))
     )
     (property "Footprint" "Package_SO:TSSOP-14_4.4x5mm_P0.65mm" (id 2) (at 71.12 180.34 0)

Commit message: 6522A(!)
Parts:
- U2, U6: value 6522 -> 6522A
Changed lines of the file:
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@@
       (effects (font (size 1.524 1.524)))
     )
-    (property "Value" "6522" (id 1) (at 205.74 76.2 0)
+    (property "Value" "6522A" (id 1) (at 205.74 76.2 0)
       (effects (font (size 1.524 1.524)))
     )
@@
       (effects (font (size 1.524 1.524)))
     )
-    (property "Value" "6522" (id 1) (at 205.74 169.545 0)
+    (property "Value" "6522A" (id 1) (at 205.74 169.545 0)
       (effects (font (size 1.524 1.524)))
     )
@@
     )
     (path "/00000000-0000-0000-0000-00005b9bfda5"
-      (reference "U2") (unit 1) (value "6522") (footprint "Package_DIP:DIP-40_W15.24mm")
+      (reference "U2") (unit 1) (value "6522A") (footprint "Package_DIP:DIP-40_W15.24mm")
     )
     (path "/8ab553b7-4763-4dd3-a825-67ce0ca1cff6"
@@
     )
     (path "/c2173ca6-7815-4e13-9854-5327be15b7fb"
-      (reference "U6") (unit 1) (value "6522") (footprint "Package_DIP:DIP-40_W15.24mm")
-    )
-  )
+      (reference "U6") (unit 1) (value "6522A") (footprint "Package_DIP:DIP-40_W15.24mm")
+    )
+  )
